Commit message: v0.5. Teleop key

File: urdf/lidar.xacro (robot description, xacro)
@@ -1,4 +1,4 @@
 <?xml version="1.0"?>
-<robot xmlns:xacro="http://ros.org/wiki/xacro">
+<robot xmlns:xacro="http://ros.org/wiki/xacro" name="lidar">
     <xacro:link name="lidar"
                 x1="0.00219031" y1="-1.11035e-18" z1="-0.0123115" mass="0.0941187"
@@ -14,5 +14,5 @@
             <pose>0 0 -0.01 0 0 0</pose>
             <visualize>true</visualize>
-            <update_rate>10</update_rate>
+            <update_rate>30</update_rate>
             <ray>
                 <scan>

File: urdf/macros.xacro (robot description, xacro)
@@ -107,3 +107,15 @@
         </joint>
     </xacro:macro>
+    <xacro:macro name="transmission" params="joint_name actuator_name">
+        <transmission name="${joint_name}_transmission">
+            <type>transmission_interface/SimpleTransmission</type>
+            <actuator name="${actuator_name}">
+                <hardwareInterface>hardware_interface/VelocityJointInterface</hardwareInterface>
+                <mechanicalReduction>1</mechanicalReduction>
+            </actuator>
+            <joint name="${joint_name}">
+                <hardwareInterface>hardware_interface/VelocityJointInterface</hardwareInterface>
+            </joint>
+        </transmission>
+    </xacro:macro>
 </robot>

File: urdf/tank.urdf.xacro (robot description, xacro)
@@ -4,4 +4,5 @@
     <xacro:include filename="chassis.xacro"/>
     <xacro:include filename="camera.xacro"/>
+    <xacro:include filename="controller.xacro"/>
     <xacro:include filename="lidar.xacro"/>
     <xacro:include filename="tracks.xacro"/>
